File: marker.kicad_pcb (KiCad board)
At the start: 2 copper layers, 21 parts, among them M1 MIC, P1 Cable, Q1 NPN, U1 MAX4475

Commit message: finish working on pcb
Parts:
- Q1: footprint Discret:TO92-123 -> SMD_Packages:SOT-23-EBC; moved to B.Cu
- moved C1 99.2 mm to (112.4, 106.0)
- moved C4 69.1 mm to (174.9, 104.8), turned to 90 degrees
- moved M1 66.4 mm to (109.5, 104.8)
- moved R5 64.5 mm to (119.1, 103.5)
- moved C7 64.2 mm to (115.6, 104.8)
- moved R7 64.2 mm to (122.6, 102.9), turned to 180 degrees
- moved L1 63.6 mm to (164.5, 105.1)
- moved C6 63.6 mm to (168.3, 104.8)
- moved R1 63.5 mm to (160.0, 106.0), turned to 90 degrees
- moved C5 63.2 mm to (164.1, 104.8)
- moved C9 62.9 mm to (127.0, 104.8)
- moved U1 62.9 mm to (133.3, 105.4)
- moved R4 62.9 mm to (123.8, 106.0)
- moved R3 62.9 mm to (120.7, 106.7)
- moved R2 62.9 mm to (157.5, 108.3)
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Routing:
- net GND: track 0.00 -> 84.8 mm
- net Net-(C8-Pad2): track 0.00 -> 41.5 mm, vias 0 -> 2
- net Net-(C1-Pad1): track 42.3 -> 55.4 mm
- net Net-(C4-Pad1): track 0.00 -> 10.9 mm
- net Net-(C6-Pad1): track 2.35 -> 12.8 mm
- net Net-(C5-Pad1): track 3.73 -> 12.7 mm
- net Net-(C7-Pad2): track 3.09 -> 10.7 mm
- net Net-(C9-Pad1): track 9.49 -> 15.0 mm
- net Net-(C8-Pad1): track 12.5 -> 7.68 mm
- net Net-(C7-Pad1): track 15.0 -> 19.0 mm
- net Net-(Q1-Pad2): track 3.49 -> 2.31 mm
- net Net-(C9-Pad2): track 3.25 -> 3.81 mm
- added copper zone on B.Cu, net GND
Other:
- board outline added: 77.2 x 6.7 mm
